Commit message: Depth sensor and grid_map

File: src/protobot_description/urdf/protobot.urdf.xacro (robot description, xacro)
@@ -81,5 +81,6 @@
 	<parent link="base_link"/>
 	<child link="camera_link"/>
-	<origin xyz="0 0.5 0.5" rpy="0 0 1.57"/>
+	<origin xyz="0 0.5 0.5" rpy="0 0 0"/>
+		<!--<origin xyz="0 0.5 0.5" rpy="0 0 1.57"/>-->
 </joint>
 <joint name="ir_joint" type="fixed">
@@ -203,5 +204,5 @@
           <stddev>0.007</stddev>
         </noise>
-      </camera>
+</camera>
       <plugin name="stereo_camera_controller" filename="libgazebo_ros_multicamera.so">
         <alwaysOn>true</alwaysOn>
@@ -211,5 +212,4 @@
         <cameraInfoTopicName>camera_info</cameraInfoTopicName>
         <frameName>camera_link</frameName>
-        <!--<rightFrameName>right_camera_optical_frame</rightFrameName>-->
         <hackBaseline>0.07</hackBaseline>
         <distortionK1>0.0</distortionK1>
@@ -218,6 +218,32 @@
         <distortionT1>0.0</distortionT1>
         <distortionT2>0.0</distortionT2>
+     </plugin>
+     </sensor>
+     <sensor type="depth" name="depth_camera">
+      <plugin name="camera_link_controller" filename="libgazebo_ros_openni_kinect.so">
+          <baseline>0.2</baseline>
+          <alwaysOn>true</alwaysOn>
+          <updateRate>1.0</updateRate>
+          <cameraName>camera</cameraName>
+          <imageTopicName>camera_gazebo/color/image_raw</imageTopicName>
+          <cameraInfoTopicName>camera_gazebo/color/camera_info</cameraInfoTopicName>
+          <depthImageTopicName>camera_gazebo/depth/image_raw</depthImageTopicName>
+          <depthImageInfoTopicName>camera_gazebo/depth/camera_info</depthImageInfoTopicName>
+	  <pointCloudTopicName>depth_camera/pointcloud</pointCloudTopicName>
+          <frameName>camera_link</frameName>
+          <pointCloudCutoff>0.5</pointCloudCutoff>
+          <pointCloudCutoffMax>3.0</pointCloudCutoffMax>
+          <distortionK1>0.00000001</distortionK1>
+          <distortionK2>0.00000001</distortionK2>
+          <distortionK3>0.00000001</distortionK3>
+          <distortionT1>0.00000001</distortionT1>
+          <distortionT2>0.00000001</distortionT2>
+          <CxPrime>0</CxPrime>
+          <Cx>0</Cx>
+          <Cy>0</Cy>
+          <focalLength>0</focalLength>
+          <hackBaseline>0</hackBaseline>
       </plugin>
-    </sensor>
+     </sensor>
   </gazebo>
 </robot>

Commit message: Fixed coordinate frames & wheel orientation

File: src/protobot_description/urdf/protobot.urdf.xacro (robot description, xacro)
@@ -70,4 +70,6 @@
 <link name="camera_link">
 </link>
+<link name="camera_link_optical">
+</link>
 <link name="ir_link">
 </link>
@@ -81,6 +83,11 @@
 	<parent link="base_link"/>
 	<child link="camera_link"/>
-	<origin xyz="0 0.5 0.5" rpy="0 0 0"/>
-		<!--<origin xyz="0 0.5 0.5" rpy="0 0 1.57"/>-->
+	<origin xyz="0 0.5 0.5" rpy="0 0 1.57"/>
+	<!--<origin xyz="0 0.5 0.5" rpy="0 0 1.57"/>-->
+</joint>
+<joint name="camera_optical_joint" type="fixed">
+	<parent link="camera_link"/>
+	<child link="camera_link_optical"/>
+	<origin xyz="0 0 0" rpy="1.57 3.14 1.57"/>
 </joint>
 <joint name="ir_joint" type="fixed">
@@ -92,5 +99,5 @@
 	<parent link="base_link"/>
 	<child link="right_wheel_link"/>
-	<origin xyz="-0.6 0.0 0" rpy="0 1.57 0"/>
+	<origin xyz="-0.6 0.0 0" rpy="3.14 1.57 0"/>
 	<axis xyz="0 0 1"/>
 </joint>
@@ -98,5 +105,5 @@
 	<parent link = "base_link"/>
 	<child link = "left_wheel_link"/>
-	<origin xyz="0.6 0 0" rpy="0 1.57 0"/>
+	<origin xyz="0.6 0 0" rpy="3.14 1.57 0"/>
 	<axis xyz="0 0 1"/>
 </joint>
@@ -231,5 +238,5 @@
           <depthImageInfoTopicName>camera_gazebo/depth/camera_info</depthImageInfoTopicName>
 	  <pointCloudTopicName>depth_camera/pointcloud</pointCloudTopicName>
-          <frameName>camera_link</frameName>
+          <frameName>camera_link_optical</frameName>
           <pointCloudCutoff>0.5</pointCloudCutoff>
           <pointCloudCutoffMax>3.0</pointCloudCutoffMax>

Commit message: Adjust elevation_mapping

File: src/protobot_description/urdf/protobot.urdf.xacro (robot description, xacro)
@@ -8,5 +8,5 @@
     </inertial>
     <visual>
-        <origin xyz="0 0 0.15"/>
+        <origin xyz="0 0 0"/>
 	<geometry>
 	    <box size="1.0 1.2 0.5"/>
@@ -83,5 +83,5 @@
 	<parent link="base_link"/>
 	<child link="camera_link"/>
-	<origin xyz="0 0.5 0.5" rpy="0 0 1.57"/>
+	<origin xyz="0 -0.5 0.5" rpy="3.1415 3.1415 1.571"/>
 	<!--<origin xyz="0 0.5 0.5" rpy="0 0 1.57"/>-->
 </joint>
@@ -89,5 +89,5 @@
 	<parent link="camera_link"/>
 	<child link="camera_link_optical"/>
-	<origin xyz="0 0 0" rpy="1.57 3.14 1.57"/>
+	<origin xyz="0 0 0" rpy="1.571 3.14 1.571"/>
 </joint>
 <joint name="ir_joint" type="fixed">
@@ -99,5 +99,5 @@
 	<parent link="base_link"/>
 	<child link="right_wheel_link"/>
-	<origin xyz="-0.6 0.0 0" rpy="3.14 1.57 0"/>
+	<origin xyz="-0.6 0.0 0" rpy="0 1.57 0"/>
 	<axis xyz="0 0 1"/>
 </joint>
@@ -105,5 +105,5 @@
 	<parent link = "base_link"/>
 	<child link = "left_wheel_link"/>
-	<origin xyz="0.6 0 0" rpy="3.14 1.57 0"/>
+	<origin xyz="0.6 0 0" rpy="0 1.57 0"/>
 	<axis xyz="0 0 1"/>
 </joint>
@@ -122,5 +122,5 @@
       <topicName>imu/data</topicName>
       <serviceName>imu_service</serviceName>
-      <gaussianNoise>0.2</gaussianNoise>
+      <gaussianNoise>0</gaussianNoise>
       <updateRate>20.0</updateRate>
     </plugin>
@@ -151,5 +151,5 @@
     <wheelAcceleration>1.0</wheelAcceleration>
     <!-- Maximum torque which the wheels can produce, in Nm, defaults to 5 Nm -->
-    <wheelTorque>5</wheelTorque>
+    <wheelTorque>20</wheelTorque>
     <!-- Topic to receive geometry_msgs/Twist message commands, defaults to `cmd_vel` -->
     <commandTopic>cmd_vel</commandTopic>
@@ -162,5 +162,4 @@
     <!-- Odometry source, 0 for ENCODER, 1 for WORLD, defaults to WORLD -->
     <odometrySource>0</odometrySource>
-    <gaussianNoise>3</gaussianNoise>
     <!-- Set to true to publish transforms for the wheel links, defaults to false -->
     <publishWheelTF>false</publishWheelTF>
@@ -239,6 +238,6 @@
 	  <pointCloudTopicName>depth_camera/pointcloud</pointCloudTopicName>
           <frameName>camera_link_optical</frameName>
-          <pointCloudCutoff>0.5</pointCloudCutoff>
-          <pointCloudCutoffMax>3.0</pointCloudCutoffMax>
+          <pointCloudCutoff>0.1</pointCloudCutoff>
+          <pointCloudCutoffMax>5</pointCloudCutoffMax>
           <distortionK1>0.00000001</distortionK1>
           <distortionK2>0.00000001</distortionK2>
