Commit message: diff drive config and integration not complete

File: src/protobot_description/urdf/rover_simple.xacro (robot description, xacro)
@@ -20,5 +20,5 @@
   </link>
   <link name="right_front_wheel"><xacro:wheel_visual_collision_inertia/></link>
-  <joint name="right_front_wheel_pivot" type="fixed">
+  <joint name="right_front_wheel_pivot" type="continuous">
     <parent link="base_link"/>
     <child link="right_front_wheel"/>
@@ -26,5 +26,5 @@
   </joint>
   <link name="right_mid_wheel"><xacro:wheel_visual_collision_inertia/></link>
-  <joint name="right_mid_wheel_pivot" type="fixed">
+  <joint name="right_mid_wheel_pivot" type="continuous">
     <parent link="base_link"/>
     <child link="right_mid_wheel"/>
@@ -32,5 +32,5 @@
   </joint>
   <link name="right_back_wheel"><xacro:wheel_visual_collision_inertia/></link>
-  <joint name="right_back_wheel_pivot" type="fixed">
+  <joint name="right_back_wheel_pivot" type="continuous">
     <parent link="base_link"/>
     <child link="right_back_wheel"/>
@@ -38,5 +38,5 @@
   </joint>
   <link name="left_front_wheel"><xacro:wheel_visual_collision_inertia/></link>
-  <joint name="left_front_wheel_pivot" type="fixed">
+  <joint name="left_front_wheel_pivot" type="continuous">
     <parent link="base_link"/>
     <child link="left_front_wheel"/>
@@ -44,5 +44,5 @@
   </joint>
   <link name="left_mid_wheel"><xacro:wheel_visual_collision_inertia/></link>
-  <joint name="left_mid_wheel_pivot" type="fixed">
+  <joint name="left_mid_wheel_pivot" type="continuous">
     <parent link="base_link"/>
     <child link="left_mid_wheel"/>
@@ -50,5 +50,5 @@
   </joint>
   <link name="left_back_wheel"><xacro:wheel_visual_collision_inertia/></link>
-  <joint name="left_back_wheel_pivot" type="fixed">
+  <joint name="left_back_wheel_pivot" type="continuous">
     <parent link="base_link"/>
     <child link="left_back_wheel"/>

Commit message: Move_base and holonomics

File: src/protobot_description/urdf/rover_simple.xacro (robot description, xacro)
@@ -69,8 +69,77 @@
     <material>Gazebo/Orange</material>
   </gazebo>
+  <link name="gps_imu_link">
+  </link>
+  <link name="camera_link">
+  </link>
+  <link name="camera_link_optical">
+  </link>
+  <joint name="gps_imu_joint" type="fixed">
+	  <parent link="base_link"/>
+	  <child link="gps_imu_link"/>
+	  <origin xyz="0 0 0.5"/>
+  </joint>
+  <joint name="camera_joint" type="fixed">
+	  <parent link="base_link"/>
+	  <child link="camera_link"/>
+	  <origin xyz="0 -0.5 0.5" rpy="3.1415 3.1415 1.571"/>
+	  <!--<origin xyz="0 0.5 0.5" rpy="0 0 1.57"/>-->
+  </joint>
+  <joint name="camera_optical_joint" type="fixed">
+	  <parent link="camera_link"/>
+	  <child link="camera_link_optical"/>
+	  <origin xyz="0 0 0" rpy="1.571 3.14 1.571"/>
+  </joint>
   <gazebo>
     <plugin filename="libgazebo_ros_control.so" name="gazebo_ros_control">
       <robotSimType>gazebo_ros_control/DefaultRobotHWSim</robotSimType>
     </plugin>
+  </gazebo>
+  <gazebo>
+	<plugin name="gps_controller" filename="libhector_gazebo_ros_gps.so">
+		<updateRate>30.0</updateRate>
+		<bodyName>gps_imu_link</bodyName>
+		<topicName>gps/fix</topicName>
+		<frameId>gps_imu_link</frameId>
+		<gaussianNoise>0</gaussianNoise>
+	</plugin>
+  </gazebo>
+  <gazebo>
+     <plugin name="imu_plugin" filename="libgazebo_ros_imu.so">
+      <alwaysOn>true</alwaysOn>
+      <bodyName>gps_imu_link</bodyName>
+      <topicName>imu/data</topicName>
+      <serviceName>imu_service</serviceName>
+      <gaussianNoise>0</gaussianNoise>
+      <updateRate>20.0</updateRate>
+    </plugin>
+  </gazebo>
+  <gazebo reference="camera_link">
+     <sensor type="depth" name="depth_camera">
+      <plugin name="camera_link_controller" filename="libgazebo_ros_openni_kinect.so">
+          <baseline>0.2</baseline>
+          <alwaysOn>true</alwaysOn>
+          <updateRate>1.0</updateRate>
+          <cameraName>camera</cameraName>
+          <imageTopicName>color/image_raw</imageTopicName>
+	  <cameraInfoTopicName>color/camera_info</cameraInfoTopicName>
+	  <depthImageTopicName>depth/image_raw</depthImageTopicName>
+	  <depthImageInfoTopicName>depth/camera_info</depthImageInfoTopicName>
+	  <pointCloudTopicName>depth/pointcloud</pointCloudTopicName>
+          <frameName>camera_link_optical</frameName>
+          <pointCloudCutoff>0.1</pointCloudCutoff>
+	  <pointCloudCutoffMax>5</pointCloudCutoffMax>
+          <distortionK1>0.00000001</distortionK1>
+          <distortionK2>0.00000001</distortionK2>
+          <distortionK3>0.00000001</distortionK3>
+          <distortionT1>0.00000001</distortionT1>
+          <distortionT2>0.00000001</distortionT2>
+          <CxPrime>0</CxPrime>
+          <Cx>0</Cx>
+          <Cy>0</Cy>
+          <focalLength>0</focalLength>
+          <hackBaseline>0</hackBaseline>
+      </plugin>
+     </sensor>
   </gazebo>
   <transmission name="left_front_trans">

Commit message: Moved realsense_ros_gazebo submodule

File: src/protobot_description/urdf/rover_simple.xacro (robot description, xacro)
@@ -91,4 +91,12 @@
 	  <origin xyz="0 0 0" rpy="1.571 3.14 1.571"/>
   </joint>
+  <xacro:include filename="$(find realsense_ros_gazebo)/xacro/tracker.xacro"/>
+  <xacro:realsense_R200 sensor_name="camera" parent_link="base_link" rate="30.0">
+    <origin rpy="0 0 0" xyz="0 0 0.5"/>
+  </xacro:realsense_R200>
+  <xacro:include filename="$(find realsense_ros_gazebo)/xacro/depthcam.xacro"/>
+  <xacro:realsense_d435 sensor_name="d435" parent_link="base_link" rate="10">
+    <origin rpy="0 0 0 " xyz="0 0 0.5"/>
+  </xacro:realsense_d435>
   <gazebo>
     <plugin filename="libgazebo_ros_control.so" name="gazebo_ros_control">

Commit message: Cameras integrated into simulated comp chassis URDF

File: src/protobot_description/urdf/rover_simple.xacro (robot description, xacro)
@@ -71,8 +71,4 @@
   <link name="gps_imu_link">
   </link>
-  <link name="camera_link">
-  </link>
-  <link name="camera_link_optical">
-  </link>
   <joint name="gps_imu_joint" type="fixed">
 	  <parent link="base_link"/>
@@ -80,19 +76,8 @@
 	  <origin xyz="0 0 0.5"/>
   </joint>
-  <joint name="camera_joint" type="fixed">
-	  <parent link="base_link"/>
-	  <child link="camera_link"/>
-	  <origin xyz="0 -0.5 0.5" rpy="3.1415 3.1415 1.571"/>
-	  <!--<origin xyz="0 0.5 0.5" rpy="0 0 1.57"/>-->
-  </joint>
-  <joint name="camera_optical_joint" type="fixed">
-	  <parent link="camera_link"/>
-	  <child link="camera_link_optical"/>
-	  <origin xyz="0 0 0" rpy="1.571 3.14 1.571"/>
-  </joint>
   <xacro:include filename="$(find realsense_ros_gazebo)/xacro/tracker.xacro"/>
-  <xacro:realsense_R200 sensor_name="camera" parent_link="base_link" rate="30.0">
+  <xacro:realsense_T265 sensor_name="camera" parent_link="base_link" rate="30.0">
     <origin rpy="0 0 0" xyz="0 0 0.5"/>
-  </xacro:realsense_R200>
+  </xacro:realsense_T265>
   <xacro:include filename="$(find realsense_ros_gazebo)/xacro/depthcam.xacro"/>
   <xacro:realsense_d435 sensor_name="d435" parent_link="base_link" rate="10">

File: src/realsense_ros_gazebo/xacro/tracker.xacro (robot description, xacro)
@@ -187,5 +187,5 @@
             <topicName>${sensor_name}/odom/sample</topicName>
             <gaussianNoise>0.001</gaussianNoise>
-            <frameName>world</frameName>
+	    <frameName>world</frameName>
             <xyzOffsets>0 0 0</xyzOffsets>
             <rpyOffsets>0 0 0</rpyOffsets>

Commit message: refined global and local costmaps and created new rviz config for displaying costmaps and paths

File: src/protobot_description/urdf/rover_simple.xacro (robot description, xacro)
@@ -71,4 +71,18 @@
   <link name="gps_imu_link">
   </link>
+  <link name="cam_link">
+</link>
+  <link name="cam_link_optical">
+</link>
+  <joint name="cam_optical_joint" type="fixed">
+	<parent link="cam_link"/>
+	<child link="cam_link_optical"/>
+	<origin xyz="0 0 0" rpy="3.14 3.14 1.571"/>
+</joint>
+  <joint name="cam_joint" type="fixed">
+	<parent link="base_link"/>
+	<child link="cam_link"/>
+	<origin xyz="0 0 0" rpy="0 0 0"/>
+</joint>
   <joint name="gps_imu_joint" type="fixed">
 	  <parent link="base_link"/>
@@ -77,14 +91,13 @@
   </joint>
   <xacro:include filename="$(find realsense_ros_gazebo)/xacro/tracker.xacro"/>
-  <xacro:realsense_T265 sensor_name="camera" parent_link="base_link" rate="30.0">
+  <xacro:realsense_T265 sensor_name="camera" parent_link="cam_link" rate="30.0">
     <origin rpy="0 0 0" xyz="0 0 0.5"/>
   </xacro:realsense_T265>
   <xacro:include filename="$(find realsense_ros_gazebo)/xacro/depthcam.xacro"/>
-  <xacro:realsense_d435 sensor_name="d435" parent_link="base_link" rate="10">
-    <origin rpy="0 0 0 " xyz="0 0 0.5"/>
+  <xacro:realsense_d435 sensor_name="d435" parent_link="cam_link" rate="10">
+    <origin rpy="0 0 0" xyz="0 0 0.5"/>
   </xacro:realsense_d435>
   <gazebo>
     <plugin filename="libgazebo_ros_control.so" name="gazebo_ros_control">
-      <robotSimType>gazebo_ros_control/DefaultRobotHWSim</robotSimType>
     </plugin>
   </gazebo>
@@ -120,5 +133,5 @@
 	  <depthImageInfoTopicName>depth/camera_info</depthImageInfoTopicName>
 	  <pointCloudTopicName>depth/pointcloud</pointCloudTopicName>
-          <frameName>camera_link_optical</frameName>
+          <frameName>cam_link_optical</frameName>
           <pointCloudCutoff>0.1</pointCloudCutoff>
 	  <pointCloudCutoffMax>5</pointCloudCutoffMax>

Commit message: Remapping to work on live hardware

File: src/protobot_description/urdf/rover_simple.xacro (robot description, xacro)
@@ -75,4 +75,5 @@
   <link name="cam_link_optical">
 </link>
+  <link name="gps"></link>
   <joint name="cam_optical_joint" type="fixed">
 	<parent link="cam_link"/>
@@ -84,4 +85,9 @@
 	<child link="cam_link"/>
 	<origin xyz="0 0 0" rpy="0 0 0"/>
+</joint>
+  <joint name="ublox_gps_joint" type="fixed">
+	<parent link="base_link"/>
+	<child link="gps"/>
+	<origin xyz="0 0 0.5"/>
 </joint>
   <joint name="gps_imu_joint" type="fixed">

Commit message: added back layers to global costmap. obstacles detection nodelet added to rtabmap launch file

File: src/protobot_description/urdf/rover_simple.xacro (robot description, xacro)
@@ -91,10 +91,10 @@
   </joint>
   <xacro:include filename="$(find realsense_ros_gazebo)/xacro/tracker.xacro"/>
-  <xacro:realsense_T265 sensor_name="camera" parent_link="cam_link" rate="30.0">
-    <origin rpy="0 0 0" xyz="0 0 0.5"/>
+  <xacro:realsense_T265 sensor_name="camera" parent_link="cam_link_optical" rate="30.0">
+    <origin rpy="0 0 1.57" xyz="0 0 0.5"/>
   </xacro:realsense_T265>
   <xacro:include filename="$(find realsense_ros_gazebo)/xacro/depthcam.xacro"/>
-  <xacro:realsense_d435 sensor_name="d435" parent_link="cam_link" rate="10">
-    <origin rpy="0 0 0" xyz="0 0 0.5"/>
+  <xacro:realsense_d435 sensor_name="d435" parent_link="cam_link_optical" rate="10">
+    <origin rpy="0 0 1.57" xyz="0 0 0.5"/>
   </xacro:realsense_d435>
   <gazebo>

Commit message: rearranged launch scheme for better hardware compat

File: src/protobot_description/urdf/rover_simple.xacro (robot description, xacro)
@@ -85,10 +85,10 @@
 	<child link="cam_link"/>
 	<origin xyz="0 0 0" rpy="0 0 0"/>
-</joint>
+  </joint>
   <joint name="ublox_gps_joint" type="fixed">
 	<parent link="base_link"/>
 	<child link="gps"/>
 	<origin xyz="0 0 0.5"/>
-</joint>
+  </joint>
   <joint name="gps_imu_joint" type="fixed">
 	  <parent link="base_link"/>

Commit message: Issue97 (#114)

File: src/protobot_description/urdf/rover_simple.xacro (robot description, xacro)
@@ -97,10 +97,10 @@
   </joint>
   <xacro:include filename="$(find realsense_ros_gazebo)/xacro/tracker.xacro"/>
-  <xacro:realsense_T265 sensor_name="camera" parent_link="cam_link" rate="30.0">
-    <origin rpy="0 0 0" xyz="0 0 0.5"/>
+  <xacro:realsense_T265 sensor_name="camera" parent_link="cam_link_optical" rate="30.0">
+    <origin rpy="0 0 1.57" xyz="0 0 0.5"/>
   </xacro:realsense_T265>
   <xacro:include filename="$(find realsense_ros_gazebo)/xacro/depthcam.xacro"/>
-  <xacro:realsense_d435 sensor_name="d435" parent_link="cam_link" rate="10">
-    <origin rpy="0 0 0" xyz="0 0 0.5"/>
+  <xacro:realsense_d435 sensor_name="d435" parent_link="cam_link_optical" rate="10">
+    <origin rpy="0 0 1.57" xyz="0 0 0.5"/>
   </xacro:realsense_d435>
   <gazebo>

Commit message: updated urdf with cam location

File: src/protobot_description/urdf/rover_simple.xacro (robot description, xacro)
@@ -79,5 +79,5 @@
 	<parent link="cam_link"/>
 	<child link="cam_link_optical"/>
-	<origin xyz="0 0 0" rpy="3.14 3.14 1.571"/>
+	<origin xyz="0.55 0 -0.1" rpy="3.14 3.14 1.571"/>
 </joint>
   <joint name="cam_joint" type="fixed">

Commit message: working navigation stack on TX2

File: src/protobot_description/urdf/rover_simple.xacro (robot description, xacro)
@@ -79,5 +79,5 @@
 	<parent link="cam_link"/>
 	<child link="cam_link_optical"/>
-	<origin xyz="0.55 0 -0.1" rpy="3.14 3.14 1.571"/>
+	<origin xyz="0 0 0" rpy="3.14 3.14 1.571"/>
 </joint>
   <joint name="cam_joint" type="fixed">
@@ -85,10 +85,10 @@
 	<child link="cam_link"/>
 	<origin xyz="0 0 0" rpy="0 0 0"/>
-  </joint>
+</joint>
   <joint name="ublox_gps_joint" type="fixed">
 	<parent link="base_link"/>
 	<child link="gps"/>
 	<origin xyz="0 0 0.5"/>
-  </joint>
+</joint>
   <joint name="gps_imu_joint" type="fixed">
 	  <parent link="base_link"/>
@@ -97,10 +97,10 @@
   </joint>
   <xacro:include filename="$(find realsense_ros_gazebo)/xacro/tracker.xacro"/>
-  <xacro:realsense_T265 sensor_name="camera" parent_link="cam_link_optical" rate="30.0">
-    <origin rpy="0 0 1.57" xyz="0 0 0.5"/>
+  <xacro:realsense_T265 sensor_name="camera" parent_link="cam_link" rate="30.0">
+    <origin rpy="0 0 0" xyz="0 0 0.5"/>
   </xacro:realsense_T265>
   <xacro:include filename="$(find realsense_ros_gazebo)/xacro/depthcam.xacro"/>
-  <xacro:realsense_d435 sensor_name="d435" parent_link="cam_link_optical" rate="10">
-    <origin rpy="0 0 1.57" xyz="0 0 0.5"/>
+  <xacro:realsense_d435 sensor_name="d435" parent_link="cam_link" rate="10">
+    <origin rpy="0 0 0" xyz="0 0 0.5"/>
   </xacro:realsense_d435>
   <gazebo>

Commit message: Remove cam_link

File: src/protobot_description/urdf/rover_simple.xacro (robot description, xacro)
@@ -71,19 +71,5 @@
   <link name="gps_imu_link">
   </link>
-  <link name="cam_link">
-</link>
-  <link name="cam_link_optical">
-</link>
   <link name="gps"></link>
-  <joint name="cam_optical_joint" type="fixed">
-	<parent link="cam_link"/>
-	<child link="cam_link_optical"/>
-	<origin xyz="0 0 0" rpy="3.14 3.14 1.571"/>
-</joint>
-  <joint name="cam_joint" type="fixed">
-	<parent link="base_link"/>
-	<child link="cam_link"/>
-	<origin xyz="0 0 0" rpy="0 0 0"/>
-</joint>
   <joint name="ublox_gps_joint" type="fixed">
 	<parent link="base_link"/>
@@ -96,4 +82,5 @@
 	  <origin xyz="0 0 0.5"/>
   </joint>
+  <!--
   <xacro:include filename="$(find realsense_ros_gazebo)/xacro/tracker.xacro"/>
   <xacro:realsense_T265 sensor_name="camera" parent_link="cam_link" rate="30.0">
@@ -104,4 +91,5 @@
     <origin rpy="0 0 0" xyz="0 0 0.5"/>
   </xacro:realsense_d435>
+-->
   <gazebo>
     <plugin filename="libgazebo_ros_control.so" name="gazebo_ros_control">

Commit message: Fix link positioning

File: src/protobot_description/urdf/rover_simple.xacro (robot description, xacro)
@@ -80,5 +80,5 @@
 	  <parent link="base_link"/>
 	  <child link="gps_imu_link"/>
-	  <origin xyz="0 0 0.5"/>
+	  <origin xyz="0 0 0"/>
   </joint>
   <!--

Commit message: Move gps link

File: src/protobot_description/urdf/rover_simple.xacro (robot description, xacro)
@@ -75,5 +75,5 @@
 	<parent link="base_link"/>
 	<child link="gps"/>
-	<origin xyz="0 0 0.5"/>
+	<origin xyz="0 0 0"/>
 </joint>
   <joint name="gps_imu_joint" type="fixed">
