Commit message: skid steering integrated using diff_drive_controller

File: src/protobot_description/urdf/macro.xacro (robot description, xacro)
@@ -42,10 +42,3 @@
   </inertial>
 </xacro:macro>
-<!--xacro:macro name="create_joints" args="prefix x y z">
-  <joint name="${prefix}_wheel_pivot" type="fixed">
-    <parent link="base_link"/>
-    <child link="${prefix}_wheel"/>
-    <origin xyz="${x} ${y} ${z}"/>
-  </joint>
-</xacro:macro-->
 </robot>

File: src/protobot_description/urdf/rover_simple.xacro (robot description, xacro)
@@ -21,19 +21,25 @@
   <link name="right_front_wheel"><xacro:wheel_visual_collision_inertia/></link>
   <joint name="right_front_wheel_pivot" type="continuous">
+    <hardwareInterface>hardware_interface/VelocityJointInterface</hardwareInterface>
     <parent link="base_link"/>
     <child link="right_front_wheel"/>
     <origin xyz="${front_wheel_forward} -${front_wheel_out} -${wheel_height}"/>
+    <axis xyz="0 1 0" />
   </joint>
   <link name="right_mid_wheel"><xacro:wheel_visual_collision_inertia/></link>
   <joint name="right_mid_wheel_pivot" type="continuous">
+    <hardwareInterface>hardware_interface/VelocityJointInterface</hardwareInterface>
     <parent link="base_link"/>
     <child link="right_mid_wheel"/>
     <origin xyz="0 -${mid_wheel_out} -${wheel_height}"/>
+    <axis xyz="0 1 0" />
   </joint>
   <link name="right_back_wheel"><xacro:wheel_visual_collision_inertia/></link>
   <joint name="right_back_wheel_pivot" type="continuous">
+    <hardwareInterface>hardware_interface/VelocityJointInterface</hardwareInterface>
     <parent link="base_link"/>
     <child link="right_back_wheel"/>
     <origin xyz="-${rear_wheel_back} -${rear_wheel_out} -${wheel_height}"/>
+    <axis xyz="0 1 0" />
   </joint>
   <link name="left_front_wheel"><xacro:wheel_visual_collision_inertia/></link>
@@ -42,19 +48,83 @@
     <child link="left_front_wheel"/>
     <origin xyz="${front_wheel_forward} ${front_wheel_out} -${wheel_height}"/>
+    <axis xyz="0 1 0" />
   </joint>
   <link name="left_mid_wheel"><xacro:wheel_visual_collision_inertia/></link>
   <joint name="left_mid_wheel_pivot" type="continuous">
+    <hardwareInterface>hardware_interface/VelocityJointInterface</hardwareInterface>
     <parent link="base_link"/>
     <child link="left_mid_wheel"/>
     <origin xyz="0 ${mid_wheel_out} -${wheel_height}"/>
+    <axis xyz="0 1 0" />
   </joint>
   <link name="left_back_wheel"><xacro:wheel_visual_collision_inertia/></link>
   <joint name="left_back_wheel_pivot" type="continuous">
+    <hardwareInterface>hardware_interface/VelocityJointInterface</hardwareInterface>
     <parent link="base_link"/>
     <child link="left_back_wheel"/>
     <origin xyz="-${rear_wheel_back} ${rear_wheel_out} -${wheel_height}"/>
+    <axis xyz="0 1 0" />
   </joint>
   <gazebo reference="base_link">
     <material>Gazebo/Orange</material>
   </gazebo>
+  <gazebo>
+    <plugin filename="libgazebo_ros_control.so" name="gazebo_ros_control">
+      <robotSimType>gazebo_ros_control/DefaultRobotHWSim</robotSimType>
+    </plugin>
+  </gazebo>
+  <transmission name="left_front_trans">
+    <type>transmission_interface/SimpleTransmission</type>
+    <actuator name="motor1">
+      <mechanicalReduction>1</mechanicalReduction>
+    </actuator>
+    <joint name="left_front_wheel_pivot">
+      <hardwareInterface>hardware_interface/VelocityJointInterface</hardwareInterface>
+    </joint>
+  </transmission>
+  <transmission name="left_middle_trans">
+    <type>transmission_interface/SimpleTransmission</type>
+    <actuator name="motor1">
+      <mechanicalReduction>1</mechanicalReduction>
+    </actuator>
+    <joint name="left_mid_wheel_pivot">
+      <hardwareInterface>hardware_interface/VelocityJointInterface</hardwareInterface>
+    </joint>
+  </transmission>
+  <transmission name="left_back_trans">
+    <type>transmission_interface/SimpleTransmission</type>
+    <actuator name="motor1">
+      <mechanicalReduction>1</mechanicalReduction>
+    </actuator>
+    <joint name="left_back_wheel_pivot">
+      <hardwareInterface>hardware_interface/VelocityJointInterface</hardwareInterface>
+    </joint>
+  </transmission>
+  <transmission name="right_front_trans">
+    <type>transmission_interface/SimpleTransmission</type>
+    <actuator name="motor1">
+      <mechanicalReduction>1</mechanicalReduction>
+    </actuator>
+    <joint name="right_front_wheel_pivot">
+      <hardwareInterface>hardware_interface/VelocityJointInterface</hardwareInterface>
+    </joint>
+  </transmission>
+  <transmission name="right_middle_trans">
+    <type>transmission_interface/SimpleTransmission</type>
+    <actuator name="motor1">
+      <mechanicalReduction>1</mechanicalReduction>
+    </actuator>
+    <joint name="right_mid_wheel_pivot">
+      <hardwareInterface>hardware_interface/VelocityJointInterface</hardwareInterface>
+    </joint>
+  </transmission>
+  <transmission name="right_back_trans">
+    <type>transmission_interface/SimpleTransmission</type>
+    <actuator name="motor1">
+      <mechanicalReduction>1</mechanicalReduction>
+    </actuator>
+    <joint name="right_back_wheel_pivot">
+      <hardwareInterface>hardware_interface/VelocityJointInterface</hardwareInterface>
+    </joint>
+  </transmission>
 </robot>

Commit message: Issue60 (#63)
* 6 wheeled urdf with gazebo and rviz working, not launched via protobot_description.launch

* diff drive config and integration not complete

* commiting what i have on laptop

* fiducial launch file

* skid steering integrated using diff_drive_controller

File: src/protobot_description/urdf/macro.xacro (robot description, xacro)
@@ -42,10 +42,3 @@
   </inertial>
 </xacro:macro>
-<!--xacro:macro name="create_joints" args="prefix x y z">
-  <joint name="${prefix}_wheel_pivot" type="fixed">
-    <parent link="base_link"/>
-    <child link="${prefix}_wheel"/>
-    <origin xyz="${x} ${y} ${z}"/>
-  </joint>
-</xacro:macro-->
 </robot>

File: src/protobot_description/urdf/rover_simple.xacro (robot description, xacro)
@@ -20,41 +20,112 @@
   </link>
   <link name="right_front_wheel"><xacro:wheel_visual_collision_inertia/></link>
-  <joint name="right_front_wheel_pivot" type="fixed">
+  <joint name="right_front_wheel_pivot" type="continuous">
+    <hardwareInterface>hardware_interface/VelocityJointInterface</hardwareInterface>
     <parent link="base_link"/>
     <child link="right_front_wheel"/>
     <origin xyz="${front_wheel_forward} -${front_wheel_out} -${wheel_height}"/>
+    <axis xyz="0 1 0" />
   </joint>
   <link name="right_mid_wheel"><xacro:wheel_visual_collision_inertia/></link>
-  <joint name="right_mid_wheel_pivot" type="fixed">
+  <joint name="right_mid_wheel_pivot" type="continuous">
+    <hardwareInterface>hardware_interface/VelocityJointInterface</hardwareInterface>
     <parent link="base_link"/>
     <child link="right_mid_wheel"/>
     <origin xyz="0 -${mid_wheel_out} -${wheel_height}"/>
+    <axis xyz="0 1 0" />
   </joint>
   <link name="right_back_wheel"><xacro:wheel_visual_collision_inertia/></link>
-  <joint name="right_back_wheel_pivot" type="fixed">
+  <joint name="right_back_wheel_pivot" type="continuous">
+    <hardwareInterface>hardware_interface/VelocityJointInterface</hardwareInterface>
     <parent link="base_link"/>
     <child link="right_back_wheel"/>
     <origin xyz="-${rear_wheel_back} -${rear_wheel_out} -${wheel_height}"/>
+    <axis xyz="0 1 0" />
   </joint>
   <link name="left_front_wheel"><xacro:wheel_visual_collision_inertia/></link>
-  <joint name="left_front_wheel_pivot" type="fixed">
+  <joint name="left_front_wheel_pivot" type="continuous">
     <parent link="base_link"/>
     <child link="left_front_wheel"/>
     <origin xyz="${front_wheel_forward} ${front_wheel_out} -${wheel_height}"/>
+    <axis xyz="0 1 0" />
   </joint>
   <link name="left_mid_wheel"><xacro:wheel_visual_collision_inertia/></link>
-  <joint name="left_mid_wheel_pivot" type="fixed">
+  <joint name="left_mid_wheel_pivot" type="continuous">
+    <hardwareInterface>hardware_interface/VelocityJointInterface</hardwareInterface>
     <parent link="base_link"/>
     <child link="left_mid_wheel"/>
     <origin xyz="0 ${mid_wheel_out} -${wheel_height}"/>
+    <axis xyz="0 1 0" />
   </joint>
   <link name="left_back_wheel"><xacro:wheel_visual_collision_inertia/></link>
-  <joint name="left_back_wheel_pivot" type="fixed">
+\
+  <joint name="left_back_wheel_pivot" type="continuous">
+    <hardwareInterface>hardware_interface/VelocityJointInterface</hardwareInterface>
     <parent link="base_link"/>
     <child link="left_back_wheel"/>
     <origin xyz="-${rear_wheel_back} ${rear_wheel_out} -${wheel_height}"/>
+    <axis xyz="0 1 0" />
   </joint>
   <gazebo reference="base_link">
     <material>Gazebo/Orange</material>
   </gazebo>
+  <gazebo>
+    <plugin filename="libgazebo_ros_control.so" name="gazebo_ros_control">
+      <robotSimType>gazebo_ros_control/DefaultRobotHWSim</robotSimType>
+    </plugin>
+  </gazebo>
+  <transmission name="left_front_trans">
+    <type>transmission_interface/SimpleTransmission</type>
+    <actuator name="motor1">
+      <mechanicalReduction>1</mechanicalReduction>
+    </actuator>
+    <joint name="left_front_wheel_pivot">
+      <hardwareInterface>hardware_interface/VelocityJointInterface</hardwareInterface>
+    </joint>
+  </transmission>
+  <transmission name="left_middle_trans">
+    <type>transmission_interface/SimpleTransmission</type>
+    <actuator name="motor1">
+      <mechanicalReduction>1</mechanicalReduction>
+    </actuator>
+    <joint name="left_mid_wheel_pivot">
+      <hardwareInterface>hardware_interface/VelocityJointInterface</hardwareInterface>
+    </joint>
+  </transmission>
+  <transmission name="left_back_trans">
+    <type>transmission_interface/SimpleTransmission</type>
+    <actuator name="motor1">
+      <mechanicalReduction>1</mechanicalReduction>
+    </actuator>
+    <joint name="left_back_wheel_pivot">
+      <hardwareInterface>hardware_interface/VelocityJointInterface</hardwareInterface>
+    </joint>
+  </transmission>
+  <transmission name="right_front_trans">
+    <type>transmission_interface/SimpleTransmission</type>
+    <actuator name="motor1">
+      <mechanicalReduction>1</mechanicalReduction>
+    </actuator>
+    <joint name="right_front_wheel_pivot">
+      <hardwareInterface>hardware_interface/VelocityJointInterface</hardwareInterface>
+    </joint>
+  </transmission>
+  <transmission name="right_middle_trans">
+    <type>transmission_interface/SimpleTransmission</type>
+    <actuator name="motor1">
+      <mechanicalReduction>1</mechanicalReduction>
+    </actuator>
+    <joint name="right_mid_wheel_pivot">
+      <hardwareInterface>hardware_interface/VelocityJointInterface</hardwareInterface>
+    </joint>
+  </transmission>
+  <transmission name="right_back_trans">
+    <type>transmission_interface/SimpleTransmission</type>
+    <actuator name="motor1">
+      <mechanicalReduction>1</mechanicalReduction>
+    </actuator>
+    <joint name="right_back_wheel_pivot">
+      <hardwareInterface>hardware_interface/VelocityJointInterface</hardwareInterface>
+    </joint>
+  </transmission>
 </robot>

Commit message: pre gui install

File: src/protobot_description/urdf/macro.xacro (robot description, xacro)
@@ -4,9 +4,9 @@
 <xacro:property name="body_width" value="0.5"/>
 <xacro:property name="body_height" value="0.2"/>
-<xacro:property name="body_mass" value="21"/>
+<xacro:property name="body_mass" value="55"/>
 <xacro:property name="wheel_radius" value="0.12"/>
 <xacro:property name="wheel_width" value="0.128"/>
 <xacro:property name="wheel_height" value="0.24"/>
-<xacro:property name="wheel_mass" value="0.5"/>
+<xacro:property name="wheel_mass" value="0.7"/>
 <xacro:property name="front_wheel_forward" value="0.4"/>
 <xacro:property name="front_wheel_out" value="0.3"/>
